File: LNS88iso.sch (KiCad schematic (older format))
At the start: 27 parts, among them CON101 AVR-ISP-6, IC101 ATTINY84-S, J101 RJ45, P101 CONN_01X02, P102 CONN_01X04, P103 CONN_01X02, P104 CONN_01X01, U101 Si8641, U102 AP1117E50, U103 AP1117E50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

Commit message: Fixed schematic symbolds
Parts:
- F101, F102: symbol F_Small -> Fuse_Small
- JP101, JP102: symbol JUMPER -> Jumper
- U102, U103: symbol AP1117E50 -> AP111750
Changed lines of the file:
@@
 EESchema Schematic File Version 2
+LIBS:LNS88iso-rescue
 LIBS:power
 LIBS:device
@@
 LIBS:valves
 LIBS:pyth
-LIBS:LNS88iso-cache
 EELAYER 25 0
 EELAYER END
@@
 Raildata
 $Comp
-L AP1117E50 U102
+L AP111750 U102
 U 1 1 55D493A5
 P 6600 1900
@@
 $EndComp
 $Comp
-L JUMPER JP102
+L Jumper JP102
 U 1 1 55DDCCFF
 P 4750 5100
@@
 $EndComp
 $Comp
-L JUMPER JP101
+L Jumper JP101
 U 1 1 55DDCF6E
 P 3850 2100
@@
 $EndComp
 $Comp
-L AP1117E50 U103
+L AP111750 U103
 U 1 1 55DDD1FF
 P 3300 1050
@@
 	4350 5100 4350 5000
 Wire Wire Line
-	3700 4600 3700 4450
+	3700 4450 3700 4600
 Wire Wire Line
 	3700 5000 3700 4900
@@
 Wire Wire Line
 	3500 2050 3500 2100
-Wire Wire Line
-	3500 2100 3550 2100
-Wire Wire Line
-	4150 2100 4250 2100
 Wire Wire Line
 	4250 2200 4200 2200
@@
 Connection ~ 7700 2350
 $Comp
-L F_Small F102
+L Fuse_Small F102
 U 1 1 55E86294
 P 7900 2700
@@
 $EndComp
 $Comp
-L F_Small F101
+L Fuse_Small F101
 U 1 1 55E86312
-P 2250 1050
-F 0 "F101" H 2210 1110 50  0000 L CNN
-F 1 "F_Small" H 2130 990 50  0000 L CNN
-F 2 "Fuse_Holders_and_Fuses:Fuse_SMD1206_HandSoldering" H 2250 1050 60  0001 C CNN
-F 3 "" H 2250 1050 60  0000 C CNN
-	1    2250 1050
-	1    0    0    -1
-$EndComp
-Wire Wire Line
-	2350 1050 3000 1050
-Wire Wire Line
-	2150 1050 2000 1050
+P 2400 1050
+F 0 "F101" H 2360 1110 50  0000 L CNN
+F 1 "F_Small" H 2280 990 50  0000 L CNN
+F 2 "Fuse_Holders_and_Fuses:Fuse_SMD1206_HandSoldering" H 2400 1050 60  0001 C CNN
+F 3 "" H 2400 1050 60  0000 C CNN
+	1    2400 1050
+	1    0    0    -1
+$EndComp
+Wire Wire Line
+	2500 1050 3000 1050
 Wire Wire Line
 	7800 2700 7700 2700
@@
 Wire Wire Line
 	3350 3500 3050 3500
+Wire Wire Line
+	4250 2100 4150 2100
+Wire Wire Line
+	3500 2100 3550 2100
+Wire Wire Line
+	2300 1050 2000 1050
 $EndSCHEMATC

Commit message: Added labels to the wires
Connections:
- net labels added: CLK, DATA, LOAD, RESET
Changed lines of the file:
@@
 Wire Wire Line
 	2300 1050 2000 1050
+Text Label 3100 3100 0    60   ~ 0
+DATA
+Text Label 3100 2800 0    60   ~ 0
+CLK
+Text Label 3100 2900 0    60   ~ 0
+LOAD
+Text Label 3100 3000 0    60   ~ 0
+RESET
 $EndSCHEMATC

Commit message: Added LED's to the unused GPIO pins of the atttiny84, silkscreen may be improved at bit
Parts:
- added D1, D2, D3: LED, LEDs:LED_0805_HandSoldering, symbol LED
- added R1, R2, R3: R, Resistors_SMD:R_0805_HandSoldering, symbol R
Connections:
- wire segments 123 -> 141
- no-connect marks 4 -> 1
Changed lines of the file:
@@
 LIBS:valves
 LIBS:pyth
+LIBS:LNS88iso-cache
 EELAYER 25 0
 EELAYER END
@@
 	-1   0    0    1
 $EndComp
-NoConn ~ 3050 3700
-NoConn ~ 3050 3800
-NoConn ~ 3050 3900
 $Comp
 L DCDC U104
@@
 $EndComp
 Wire Wire Line
-	4550 1100 4550 1050
+	4550 1050 4550 1150
 Wire Wire Line
 	4550 1050 4450 1050
 Connection ~ 4050 1050
 Wire Wire Line
-	8250 1950 8250 1900
+	8250 1900 8250 2000
 Wire Wire Line
 	8250 1900 8150 1900
@@
 Text Label 3100 3000 0    60   ~ 0
 RESET
+Wire Wire Line
+	4550 1500 4550 1450
+Wire Wire Line
+	8250 2350 8250 2300
+$Comp
+L R R1
+U 1 1 5996962B
+P 2950 4500
+F 0 "R1" V 3030 4500 50  0000 C CNN
+F 1 "R" V 2950 4500 50  0000 C CNN
+F 2 "Resistors_SMD:R_0805_HandSoldering" V 2880 4500 50  0001 C CNN
+F 3 "" H 2950 4500 50  0000 C CNN
+	1    2950 4500
+	1    0    0    -1
+$EndComp
+$Comp
+L R R2
+U 1 1 599696A6
+P 3100 4500
+F 0 "R2" V 3180 4500 50  0000 C CNN
+F 1 "R" V 3100 4500 50  0000 C CNN
+F 2 "Resistors_SMD:R_0805_HandSoldering" V 3030 4500 50  0001 C CNN
+F 3 "" H 3100 4500 50  0000 C CNN
+	1    3100 4500
+	1    0    0    -1
+$EndComp
+$Comp
+L R R3
+U 1 1 59969712
+P 3250 4500
+F 0 "R3" V 3330 4500 50  0000 C CNN
+F 1 "R" V 3250 4500 50  0000 C CNN
+F 2 "Resistors_SMD:R_0805_HandSoldering" V 3180 4500 50  0001 C CNN
+F 3 "" H 3250 4500 50  0000 C CNN
+	1    3250 4500
+	1    0    0    -1
+$EndComp
+$Comp
+L LED D1
+U 1 1 59969781
+P 2950 4850
+F 0 "D1" H 3050 4800 50  0000 C CNN
+F 1 "LED" H 2950 4750 50  0001 C CNN
+F 2 "LEDs:LED_0805_HandSoldering" H 2950 4850 50  0001 C CNN
+F 3 "" H 2950 4850 50  0000 C CNN
+	1    2950 4850
+	0    -1   -1   0
+$EndComp
+$Comp
+L LED D2
+U 1 1 599697FF
+P 3100 4850
+F 0 "D2" H 3200 4800 50  0000 C CNN
+F 1 "LED" H 3100 4750 50  0001 C CNN
+F 2 "LEDs:LED_0805_HandSoldering" H 3100 4850 50  0001 C CNN
+F 3 "" H 3100 4850 50  0000 C CNN
+	1    3100 4850
+	0    -1   -1   0
+$EndComp
+$Comp
+L LED D3
+U 1 1 59969881
+P 3250 4850
+F 0 "D3" H 3350 4800 50  0000 C CNN
+F 1 "LED" H 3250 4750 50  0000 C CNN
+F 2 "LEDs:LED_0805_HandSoldering" H 3250 4850 50  0001 C CNN
+F 3 "" H 3250 4850 50  0000 C CNN
+	1    3250 4850
+	0    -1   -1   0
+$EndComp
+Wire Wire Line
+	3250 4700 3250 4650
+Wire Wire Line
+	3100 4700 3100 4650
+Wire Wire Line
+	2950 4700 2950 4650
+Wire Wire Line
+	2950 4100 2950 4350
+Wire Wire Line
+	2950 4100 3050 4100
+Wire Wire Line
+	3050 4100 3050 3900
+Wire Wire Line
+	3050 3800 3100 3800
+Wire Wire Line
+	3100 3800 3100 4350
+Wire Wire Line
+	3250 4350 3250 4100
+Wire Wire Line
+	3250 4100 3150 4100
+Wire Wire Line
+	3150 4100 3150 3700
+Wire Wire Line
+	3150 3700 3050 3700
+Wire Wire Line
+	2950 5000 2950 5100
+Wire Wire Line
+	2950 5100 3250 5100
+Wire Wire Line
+	3100 5000 3100 5150
+Wire Wire Line
+	3250 5100 3250 5000
+Connection ~ 3100 5100
+$Comp
+L GND #PWR034
+U 1 1 5996A9D2
+P 3100 5150
+F 0 "#PWR034" H 3100 4900 50  0001 C CNN
+F 1 "GND" H 3100 5000 50  0000 C CNN
+F 2 "" H 3100 5150 50  0000 C CNN
+F 3 "" H 3100 5150 50  0000 C CNN
+	1    3100 5150
+	1    0    0    -1
+$EndComp
 $EndSCHEMATC

Commit message: Update to Kicad 5.1
Parts:
- C101, C102, C106, C107: symbol CP -> Device:CP
- C103, C104, C105: symbol C -> Device:C
- CON101: symbol AVR-ISP-6 -> Connector:AVR-ISP-6
- D1, D101, D102, D2, D3: symbol LED -> Device:LED
- F101, F102: symbol Fuse_Small -> Device:Fuse_Small
- IC101: symbol ATTINY84-S -> MCU_Microchip_ATtiny:ATtiny84-20SSU
- J101: symbol RJ45 -> LNS88iso-rescue:RJ45
- JP101, JP102: symbol Jumper -> Device:Jumper
- P101, P103: symbol CONN_01X02 -> Connector_Generic:Conn_01x02
- P102: symbol CONN_01X04 -> Connector_Generic:Conn_01x04
- P104: symbol CONN_01X01 -> Connector_Generic:Conn_01x01
- R1, R101, R102, R103, R2, R3: symbol R -> Device:R
- U101: symbol Si8641 -> pyth:Si8641
- U102, U103: symbol AP111750 -> Regulator_Linear:AP1117-50
- U104: symbol DCDC -> pyth:DCDC
Connections:
- wire segments 141 -> 177
