File: LNS88iso.kicad_pcb (KiCad board)
At the start: 2 copper layers, 50 x 50 mm, 38 parts, among them CON101 AVR-ISP-6, IC101 ATTINY84-S, J101 RJ45, P101 CONN_01X02, P102 CONN_01X04, P103 CONN_01X02, P104 CONN_01X01, U101 Si8641, U102 AP1117E50, U103 AP1117E50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

Commit message: Kicad updates
Other:
- net class Default removed
- net class Power removed
